File: wah.kicad_pcb (KiCad board)
At the start: 4 copper layers, 99.1 x 54.5 mm, 34 parts, among them J3 Barrel_Jack_Switch, J4 In, J5 Out, SW2 SW_Push_3PDT, U1 L78L05_TO92, U2 TL072

Commit message: improve pcb
Parts:
- C1, C10, C11, C12, C3, C4, C5, C6, C7, C8, C9: footprint Capacitor_THT:C_Rect_L4.6mm_W2.0mm_P2.50mm_MKS02_FKP02 -> Capacitor_THT:C_Rect_L7.0mm_W2.5mm_P5.00mm
- C2: footprint Capacitor_THT:CP_Radial_D5.0mm_P2.50mm -> Capacitor_THT:C_Rect_L7.0mm_W2.5mm_P5.00mm
- R1, R2, R3, R4, R5, R6, R7, R8, R9: footprint Resistor_THT:R_Axial_DIN0207_L6.3mm_D2.5mm_P10.16mm_Horizontal -> Resistor_THT:R_Axial_DIN0207_L6.3mm_D2.5mm_P7.62mm_Horizontal
- moved C1 12.9 mm to (74.8, 101.9), turned to -90 degrees
- moved R3 10.2 mm to (124.5, 85.1)
- moved D1 8.98 mm to (76.8, 97.7), turned to 180 degrees
- moved C5 7.86 mm to (79.7, 101.9), turned to -90 degrees
- moved C2 7.75 mm to (70.0, 101.9)
- moved C6 7.32 mm to (117.3, 107.6)
- moved R4 6.98 mm to (86.1, 77.4)
- moved C9 6.94 mm to (86.1, 81.9), turned to -90 degrees
- moved C10 6.85 mm to (124.5, 71.8)
- moved U2 6.38 mm to (119.6, 92.4)
- moved C4 6.26 mm to (89.3, 101.9), turned to -90 degrees
- moved C12 5.98 mm to (113.3, 79.6)
- moved C7 5.58 mm to (117.3, 102.3)
- moved R8 5.21 mm to (119.6, 74.7)
- moved R2 4.95 mm to (124.5, 104.6)
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Routing:
- net Net-(U1-VO): track 0.00 -> 87.9 mm
- net /FX_OUT: track 0.00 -> 59.2 mm
- net /FX_IN: track 0.00 -> 55.4 mm
- net Net-(U2B-+): track 0.00 -> 31.3 mm
- net /AUDIO_IN: track 0.00 -> 27.6 mm
- net Net-(U2A-+): track 0.00 -> 19.0 mm
- net Net-(U2B--): track 0.00 -> 18.2 mm
- net /POT1: track 0.00 -> 16.1 mm
- net Net-(C7-Pad2): track 0.00 -> 13.2 mm
- net /POT2: track 0.00 -> 12.4 mm
- net Net-(D1-A): track 0.00 -> 11.0 mm
- net Net-(C10-Pad1): track 0.00 -> 10.5 mm
- net Net-(C12-Pad1): track 0.00 -> 5.44 mm
- net Net-(SW2-A-Pad1): track 0.00 -> 5.30 mm
- net /AUDIO_OUT: track 0.00 -> 4.71 mm
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Other:
- board text added: "Vintage 1951 NOS ElectroSmith Daisy"

Commit message: improve pcb
Parts:
- added GND1: ~, TestPoint:TestPoint_THTPad_1.5x1.5mm_Drill0.7mm, F.Cu at (140.3, 90.9)
- added GND2: ~, TestPoint:TestPoint_THTPad_1.5x1.5mm_Drill0.7mm, F.Cu at (140.3, 96.0)
- added TP_IN1: TestPoint, TestPoint:TestPoint_THTPad_1.5x1.5mm_Drill0.7mm, F.Cu at (135.2, 96.1)
- added TP_OUT1: TestPoint, TestPoint:TestPoint_THTPad_1.5x1.5mm_Drill0.7mm, F.Cu at (135.2, 90.9)
- moved R9 9.75 mm to (150.9, 71.7), turned to 90 degrees
- moved U2 5.14 mm to (83.9, 96.0), turned to 0 degrees
- moved C10 4.30 mm to (87.4, 86.0)
- moved G*** 2.52 mm to (159.1, 102.8)
- moved A1 1.00 mm to (107.9, 106.7)
- moved C5 1.00 mm to (88.3, 101.9)
- moved C4 0.75 mm to (83.7, 101.9)
- moved C8 0.50 mm to (79.2, 101.9)
- moved C7 0.25 mm to (74.6, 101.9)
- moved RV2 0.16 mm to (80.6, 66.0)
- renumbered C10 to C1, C9 to C10, C7 to C11, C8 to C12, C11 to C2, C2 to C3, C3 to C4, C4 to C5, C12 to C6, C1 to C7, C5 to C8, C6 to C9, J3 to J1, J4 to J2, J5 to J3, R6 to R1, R7 to R2, R8 to R3, R9 to R4, R4 to R5, R5 to R6, R2 to R7, R3 to R8, R1 to R9, SW2 to SW1, U2 to U1, U1 to U2
Routing:
- net /FX_OUT: track 59.2 -> 66.0 mm
- net Net-(R9-Pad1): track 7.87 -> 13.7 mm
- net /FX_IN: track 55.4 -> 60.7 mm
- net Net-(U1C-V+): track 87.9 -> 83.0 mm
- net Net-(D2-A): track 7.97 -> 4.64 mm
- net /AUDIO_IN: track 27.6 -> 28.7 mm
Other:
- board text added: "Wah version 0.2"
- board text removed: "Wah V0.1"
