File: hardware/wah.kicad_pcb (KiCad board)
At the start: 4 copper layers, 99.1 x 54.5 mm, 32 parts, among them J1 Barrel_Jack_Switch, J2 In, J3 Out, SW1 SW_Push_3PDT, U1 TL072, U2 L78L05_TO92

Commit message: improve layout
Parts:
- moved C8 11.6 mm to (89.6, 85.1), turned to 0 degrees
- moved C6 11.5 mm to (89.6, 72.3)
- moved C4 11.5 mm to (89.6, 75.9)
- moved C9 8.23 mm to (89.6, 80.5), turned to 0 degrees
- moved C1 5.50 mm to (99.8, 55.6), turned to 90 degrees
- moved C2 3.19 mm to (99.8, 59.2)
- moved C5 3.10 mm to (99.8, 72.8)
- moved C10 3.00 mm to (99.8, 76.4)
Routing:
- net Net-(C5-Pad1): track 54.3 -> 73.5 mm
- net Net-(U1C-V+): track 91.2 -> 75.2 mm
- net /AUDIO_OUT: track 10.4 -> 19.2 mm
- net Net-(U1A-+): track 50.3 -> 57.9 mm
- net Net-(C9-Pad2): track 37.7 -> 32.5 mm
- net Net-(C1-Pad1): track 17.3 -> 12.6 mm
- net /POT1: track 37.3 -> 35.0 mm
- net Net-(U1B-+): track 41.4 -> 42.6 mm
- net /AUDIO_IN: track 29.3 -> 29.8 mm
Other:
- board text added: "Wah version 0.7"
- board text removed: "Wah version 0.6"
