File: hardware/wah.kicad_sch (KiCad schematic)
At the start: 36 parts, among them J1 Barrel_Jack_Switch, J2 In, J3 Out, SW1 SW_Push_3PDT, U1 TL072, U2 L78L05_TO92

Commit message: create new folders
Parts:
- removed GND1, GND2: ~, TestPoint:TestPoint_THTPad_1.5x1.5mm_Drill0.7mm, symbol Connector:TestPoint
- removed TP_IN1, TP_OUT1: TestPoint, TestPoint:TestPoint_THTPad_1.5x1.5mm_Drill0.7mm, symbol Connector:TestPoint

Commit message: fix footprints
Parts:
- C11, C12, C2, C6: footprint Capacitor_THT:C_Rect_L7.0mm_W2.5mm_P5.00mm -> Capacitor_THT:C_Rect_L7.0mm_W4.5mm_P5.00mm
- C13, C3: footprint Capacitor_THT:CP_Radial_D6.3mm_P2.50mm -> Capacitor_THT:CP_Radial_D5.0mm_P2.50mm
Changed lines of the file:
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@@
 	(title_block
 		(title "Wah")
-		(date "2025-11-11")
-		(rev "0.4.3")
+		(date "2025-11-13")
+		(rev "0.6")
 		(company "KnightHill Engineering")
 	)
@@
 			)
 		)
-		(property "Footprint" "Capacitor_THT:C_Rect_L7.0mm_W2.5mm_P5.00mm"
+		(property "Footprint" "Capacitor_THT:C_Rect_L7.0mm_W4.5mm_P5.00mm"
 			(at 274.0152 74.93 0)
 			(effects
@@
 			)
 		)
-		(property "Footprint" "Capacitor_THT:C_Rect_L7.0mm_W2.5mm_P5.00mm"
+		(property "Footprint" "Capacitor_THT:C_Rect_L7.0mm_W4.5mm_P5.00mm"
 			(at 193.04 63.8048 0)
 			(effects
@@
 			)
 		)
-		(property "Footprint" "Capacitor_THT:C_Rect_L7.0mm_W2.5mm_P5.00mm"
+		(property "Footprint" "Capacitor_THT:C_Rect_L7.0mm_W4.5mm_P5.00mm"
 			(at 142.24 61.2648 0)
 			(effects
@@
 			)
 		)
-		(property "Footprint" "Capacitor_THT:CP_Radial_D6.3mm_P2.50mm"
+		(property "Footprint" "Capacitor_THT:CP_Radial_D5.0mm_P2.50mm"
 			(at 143.2052 237.49 0)
 			(effects
@@
 			)
 		)
-		(property "Footprint" "Capacitor_THT:CP_Radial_D6.3mm_P2.50mm"
+		(property "Footprint" "Capacitor_THT:CP_Radial_D5.0mm_P2.50mm"
 			(at 247.3452 237.49 0)
 			(effects
@@
 			)
 		)
-		(property "Footprint" "Capacitor_THT:C_Rect_L7.0mm_W2.5mm_P5.00mm"
+		(property "Footprint" "Capacitor_THT:C_Rect_L7.0mm_W4.5mm_P5.00mm"
 			(at 252.73 63.8048 0)
 			(effects

Commit message: rearrange pcb
Parts:
- removed C4, C5: 100n, Capacitor_THT:C_Rect_L7.0mm_W2.5mm_P5.00mm, symbol Device:C
Other:
- moved on the sheet: C13, C7, C8, R5, R6, U1C, U2

Commit message: rename resources
Parts:
- renumbered C12 to C10, C7 to C4, C6 to C5, C8 to C6, C13 to C7, C9 to C8, C11 to C9
Changed lines of the file:
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@@
 		(dnp no)
 		(fields_autoplaced yes)
-		(property "Reference" "#PWR022"
+		(property "Reference" "#PWR020"
 			(at 256.54 137.16 0)
 			(effects
@@
 			(project "roundup"
 				(path "/93d00cbf-8e4b-443f-bc57-0c283a060166"
-					(reference "#PWR022")
+					(reference "#PWR020")
 					(unit 1)
 				)
@@
 		(dnp no)
 		(fields_autoplaced yes)
-		(property "Reference" "#PWR013"
+		(property "Reference" "#PWR09"
 			(at 167.64 248.92 0)
 			(effects
@@
 			(project "roundup"
 				(path "/93d00cbf-8e4b-443f-bc57-0c283a060166"
-					(reference "#PWR013")
+					(reference "#PWR09")
 					(unit 1)
 				)
@@
 		(dnp no)
 		(fields_autoplaced yes)
-		(property "Reference" "#PWR018"
+		(property "Reference" "#PWR016"
 			(at 199.39 248.92 0)
 			(effects
@@
 			(project "roundup"
 				(path "/93d00cbf-8e4b-443f-bc57-0c283a060166"
-					(reference "#PWR018")
+					(reference "#PWR016")
 					(unit 1)
 				)
@@
 		(dnp no)
 		(fields_autoplaced yes)
-		(property "Reference" "#PWR019"
+		(property "Reference" "#PWR017"
 			(at 217.17 248.92 0)
 			(effects
@@
 			(project "wah"
 				(path "/93d00cbf-8e4b-443f-bc57-0c283a060166"
-					(reference "#PWR019")
+					(reference "#PWR017")
 					(unit 1)
 				)
@@
 		(dnp no)
 		(fields_autoplaced yes)
-		(property "Reference" "C7"
+		(property "Reference" "C4"
 			(at 182.88 232.4099 0)
 			(effects
@@
 			(project "roundup"
 				(path "/93d00cbf-8e4b-443f-bc57-0c283a060166"
-					(reference "C7")
+					(reference "C4")
 					(unit 1)
 				)
@@
 		(dnp no)
 		(fields_autoplaced yes)
-		(property "Reference" "#PWR020"
+		(property "Reference" "#PWR019"
 			(at 240.03 83.82 0)
 			(effects
@@
 			(project ""
 				(path "/93d00cbf-8e4b-443f-bc57-0c283a060166"
-					(reference "#PWR020")
+					(reference "#PWR019")
 					(unit 1)
 				)
@@
 		(dnp no)
 		(fields_autoplaced yes)
-		(property "Reference" "C12"
+		(property "Reference" "C10"
 			(at 276.86 69.8499 0)
 			(effects
@@
 			(project ""
 				(path "/93d00cbf-8e4b-443f-bc57-0c283a060166"
-					(reference "C12")
+					(reference "C10")
 					(unit 1)
 				)
@@
 		(dnp no)
 		(fields_autoplaced yes)
-		(property "Reference" "C6"
+		(property "Reference" "C5"
 			(at 189.23 57.15 90)
 			(effects
@@
 			(project ""
 				(path "/93d00cbf-8e4b-443f-bc57-0c283a060166"
-					(reference "C6")
+					(reference "C5")
 					(unit 1)
 				)
@@
 		(dnp no)
 		(fields_autoplaced yes)
-		(property "Reference" "#PWR024"
+		(property "Reference" "#PWR022"
 			(at 273.05 83.82 0)
 			(effects
@@
 			(project "wah"
 				(path "/93d00cbf-8e4b-443f-bc57-0c283a060166"
-					(reference "#PWR024")
+					(reference "#PWR022")
 					(unit 1)
 				)
@@
 		(dnp no)
 		(fields_autoplaced yes)
-		(property "Reference" "#PWR026"
+		(property "Reference" "#PWR024"
 			(at 320.04 151.13 0)
 			(effects
@@
 			(project "roundup"
 				(path "/93d00cbf-8e4b-443f-bc57-0c283a060166"
-					(reference "#PWR026")
+					(reference "#PWR024")
 					(unit 1)
 				)
@@
 		(dnp no)
 		(fields_autoplaced yes)
-		(property "Reference" "#PWR023"
+		(property "Reference" "#PWR021"
 			(at 256.54 151.13 0)
 			(effects
@@
 			(project "roundup"
 				(path "/93d00cbf-8e4b-443f-bc57-0c283a060166"
-					(reference "#PWR023")
+					(reference "#PWR021")
 					(unit 1)
 				)
@@
 		(dnp no)
 		(fields_autoplaced yes)
-		(property "Reference" "#PWR016"
+		(property "Reference" "#PWR015"
 			(at 198.12 83.82 0)
 			(effects
@@
 			(project "wah"
 				(path "/93d00cbf-8e4b-443f-bc57-0c283a060166"
-					(reference "#PWR016")
+					(reference "#PWR015")
 					(unit 1)
 				)
@@
 		(dnp no)
 		(fields_autoplaced yes)
-		(property "Reference" "#PWR021"
+		(property "Reference" "#PWR018"
 			(at 231.14 248.92 0)
 			(effects
@@
 			(project "wah"
 				(path "/93d00cbf-8e4b-443f-bc57-0c283a060166"
-					(reference "#PWR021")
+					(reference "#PWR018")
 					(unit 1)
 				)
@@
 		(dnp no)
 		(fields_autoplaced yes)
-		(property "Reference" "C9"
+		(property "Reference" "C8"
 			(at 243.84 69.8499 0)
 			(effects
@@
 			(project ""
 				(path "/93d00cbf-8e4b-443f-bc57-0c283a060166"
-					(reference "C9")
+					(reference "C8")
 					(unit 1)
 				)
@@
 		(dnp no)
 		(fields_autoplaced yes)
-		(property "Reference" "C13"
+		(property "Reference" "C7"
 			(at 234.95 231.5209 0)
 			(effects
@@
 			(project "wah"
 				(path "/93d00cbf-8e4b-443f-bc57-0c283a060166"
-					(reference "C13")
+					(reference "C7")
 					(unit 1)
 				)
@@
 		(dnp no)
 		(fields_autoplaced yes)
-		(property "Reference" "#PWR017"
+		(property "Reference" "#PWR014"
 			(at 189.23 248.92 0)
 			(effects
@@
 			(project "roundup"
 				(path "/93d00cbf-8e4b-443f-bc57-0c283a060166"
-					(reference "#PWR017")
+					(reference "#PWR014")
 					(unit 1)
 				)
@@
 		(on_board yes)
 		(dnp no)
-		(property "Reference" "#PWR014"
+		(property "Reference" "#PWR013"
 			(at 185.42 120.65 0)
 			(effects
@@
 			(project "flip-nopower"
 				(path "/93d00cbf-8e4b-443f-bc57-0c283a060166"
-					(reference "#PWR014")
+					(reference "#PWR013")
 					(unit 1)
 				)
@@
 		(dnp no)
 		(fields_autoplaced yes)
-		(property "Reference" "#PWR025"
+		(property "Reference" "#PWR023"
 			(at 284.48 148.59 0)
 			(effects
@@
 			(project "roundup"
 				(path "/93d00cbf-8e4b-443f-bc57-0c283a060166"
-					(reference "#PWR025")
+					(reference "#PWR023")
 					(unit 1)
 				)
@@
 		(dnp no)
 		(fields_autoplaced yes)
-		(property "Reference" "C8"
+		(property "Reference" "C6"
 			(at 203.2 232.4099 0)
 			(effects
@@
 			(project "roundup"
 				(path "/93d00cbf-8e4b-443f-bc57-0c283a060166"
-					(reference "C8")
+					(reference "C6")
 					(unit 1)
 				)
@@
 		(dnp no)
 		(fields_autoplaced yes)
-		(property "Reference" "#PWR015"
+		(property "Reference" "#PWR010"
 			(at 179.07 248.92 0)
 			(effects
@@
 			(project "roundup"
 				(path "/93d00cbf-8e4b-443f-bc57-0c283a060166"
-					(reference "#PWR015")
+					(reference "#PWR010")
 					(unit 1)
 				)
@@
 		(dnp no)
 		(fields_autoplaced yes)
-		(property "Reference" "C11"
+		(property "Reference" "C9"
 			(at 248.92 57.15 90)
 			(effects
@@
 			(project ""
 				(path "/93d00cbf-8e4b-443f-bc57-0c283a060166"
-					(reference "C11")
+					(reference "C9")
 					(unit 1)
 				)

Commit message: pcb
Parts:
- added H1, H2: MountingHole_Pad, MountingHole:MountingHole_3.2mm_M3_Pad, symbol Mechanical:MountingHole_Pad
- added J4: Conn_01x08_Pin, Connector_PinHeader_2.54mm:PinHeader_1x08_P2.54mm_Vertical, symbol Connector:Conn_01x08_Pin
- added RV3, RV4: 10k, Potentiometer_THT:Potentiometer_Runtron_RM-065_Vertical, symbol Device:R_Potentiometer
- added SW2: SW_DIP_x04, Button_Switch_THT:SW_DIP_SPSTx04_Slide_9.78x12.34mm_W7.62mm_P2.54mm, symbol Switch:SW_DIP_x04
- RV1, RV2: footprint CustomFootprints:Potentiometer_uxcel_9mm_Single_Vertical -> Potentiometer_THT:Potentiometer_Runtron_RM-065_Vertical
Connections:
- net +9V: now also J4.2 (Pin_2)
- net FX_IN: now also J4.5 (Pin_5)
- net FX_OUT: now also J4.6 (Pin_6)
- net GND: now also H1.1, H2.1, J4.1 (Pin_1), RV3.1, RV4.1, SW2.5, SW2.6, SW2.7, SW2.8
- net POT1: now also A1.22 (ADC_0); no longer A1.24 (ADC_2)
- net VDD: now also RV3.3, RV4.3
- net J_IN: now reaches J2.T, SW1.2 (B)
- net J_IN: now also J4.3 (Pin_3)
- net J_OUT: now reaches J3.T, SW1.5 (B)
- net J_OUT: now also J4.4 (Pin_4)
- net POT4: now reaches A1.25 (ADC_3)
- net POT4: now also RV4.2
- net SW1: now reaches A1.27 (ADC_5)
- net SW1: now also SW2.1
- net SW2: now reaches A1.28 (ADC_6)
- net SW2: now also SW2.2
- net SW3: now reaches A1.29 (DAC_OUT2)
- net SW3: now also SW2.3
- net SW4: now reaches A1.30 (DAC_OUT1)
- net SW4: now also SW2.4
- new net POT3: A1.24 (ADC_2), RV3.2
- no-connect marks 34 -> 30
Other:
- moved on the sheet: RV1, RV2

Commit message: pcb changes
Parts:
- removed D2: LED, LED_THT:LED_D5.0mm, symbol Device:LED
- removed R9: R, Resistor_THT:R_Axial_DIN0207_L6.3mm_D2.5mm_P7.62mm_Horizontal, symbol Device:R
- removed SW1: SW_Push_3PDT, CustomFootprints:Switches_Stomp_Switch_3PDT, symbol CustomSymbols:SW_Push_3PDT
- added D3: LED, LED_THT:LED_D5.0mm, symbol Device:LED
- added J5: Conn_01x08_Pin, Connector_PinHeader_2.54mm:PinHeader_1x08_P2.54mm_Vertical, symbol Connector:Conn_01x08_Pin
- added R10: R, Resistor_THT:R_Axial_DIN0207_L6.3mm_D2.5mm_P7.62mm_Horizontal, symbol Device:R
- added SW3: SW_Push_3PDT, CustomFootprints:Switches_Stomp_Switch_3PDT, symbol CustomSymbols:SW_Push_3PDT
Connections:
- net GND: now also D3.1 (K), J5.1 (Pin_1)
- net LED: now reaches J4.7 (Pin_7)
- net LED: now also R10.1
- new net: D3.2 (A), R10.2
- new net: SW3.1 (A), SW3.4 (A)
- new net: J5.3 (Pin_3), SW3.2 (B)
- new net: J5.5 (Pin_5), SW3.3 (C)
- new net: J5.4 (Pin_4), SW3.5 (B)
- new net: J5.6 (Pin_6), SW3.6 (C)
- new net: J5.2 (Pin_2), SW3.8 (B)
- new net: J5.7 (Pin_7), SW3.9 (C)
Other:
- moved on the sheet: J4
