File: hardware/switch/switch.kicad_pcb (KiCad board)
At the start: 2 copper layers, 26.4 x 17 mm, 2 parts, among them J2 Conn_01x06_Pin, SW1 SW_Push_3PDT

Commit message: remove pot 4
Other:
- outline, holes or cut-outs redrawn
Changed lines of the file:
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@@
 		(sheetname "/")
 		(sheetfile "switch.kicad_sch")
-		(attr through_hole)
+		(attr through_hole exclude_from_pos_files exclude_from_bom)
 		(fp_line
 			(start -9.8 -8.5)
@@
 		(sheetname "/")
 		(sheetfile "switch.kicad_sch")
-		(attr through_hole)
+		(attr through_hole exclude_from_pos_files exclude_from_bom)
 		(fp_line
 			(start -1.38 -1.38)
@@
 		)
 	)
-	(gr_rect
-		(start 115.54 93.285)
-		(end 141.9 110.285)
-		(stroke
-			(width 0.1)
-			(type default)
-		)
-		(fill no)
-		(layer "Edge.Cuts")
-	)
+	(gr_arc
+		(start 116.54 110.285)
+		(mid 115.832893 109.992107)
+		(end 115.54 109.285)
+		(stroke
+			(width 0.1)
+			(type default)
+		)
+		(layer "Edge.Cuts")
+	)
+	(gr_line
+		(start 115.54 109.285)
+		(end 115.54 94.285)
+		(stroke
+			(width 0.1)
+			(type default)
+		)
+		(layer "Edge.Cuts")
+	)
+	(gr_line
+		(start 116.54 93.285)
+		(end 140.9 93.285)
+		(stroke
+			(width 0.1)
+			(type default)
+		)
+		(layer "Edge.Cuts")
+	)
+	(gr_arc
+		(start 115.54 94.285)
+		(mid 115.832893 93.577893)
+		(end 116.54 93.285)
+		(stroke
+			(width 0.1)
+			(type default)
+		)
+		(layer "Edge.Cuts")
+	)
+	(gr_line
+		(start 140.9 110.285)
+		(end 116.54 110.285)
+		(stroke
+			(width 0.1)
+			(type default)
+		)
+		(layer "Edge.Cuts")
+	)
+	(gr_arc
+		(start 140.9 93.285)
+		(mid 141.607107 93.577893)
+		(end 141.9 94.285)
+		(stroke
+			(width 0.1)
+			(type default)
+		)
+		(layer "Edge.Cuts")
+	)
+	(gr_line
+		(start 141.9 94.285)
+		(end 141.9 109.285)
+		(stroke
+			(width 0.1)
+			(type default)
+		)
+		(layer "Edge.Cuts")
+	)
+	(gr_arc
+		(start 141.9 109.285)
+		(mid 141.607107 109.992107)
+		(end 140.9 110.285)
+		(stroke
+			(width 0.1)
+			(type default)
+		)
+		(layer "Edge.Cuts")
+	)
