File: hardware/crybaby/wah.kicad_sch (KiCad schematic)
At the start: 37 parts, among them J1 Barrel_Jack_Switch, J2 In, J3 Out, J4 Conn_01x08_Pin, J5 Conn_01x08_Pin, SW2 SW_DIP_x04, SW3 SW_Push_3PDT, U1 TL072, U2 L78L05_TO92

Commit message: major rearrangement
Parts:
- removed J4, J5: Conn_01x08_Pin, Connector_PinHeader_2.54mm:PinHeader_1x08_P2.54mm_Vertical, symbol Connector:Conn_01x08_Pin
- removed SW3: SW_Push_3PDT, CustomFootprints:Switches_Stomp_Switch_3PDT, symbol CustomSymbols:SW_Push_3PDT
- added J4: Conn_01x06_Pin, Connector_PinHeader_2.54mm:PinHeader_1x06_P2.54mm_Vertical, symbol Connector:Conn_01x06_Pin
- added J5: Conn_01x03_Pin, Connector_PinHeader_2.54mm:PinHeader_1x03_P2.54mm_Vertical, symbol Connector:Conn_01x03_Pin
- renumbered D3 to D2, R10 to R8, R8 to R9, SW2 to SW1
Connections:
- net +9V: now also J4.1 (Pin_1)
- net FX_IN: now also J4.4 (Pin_4)
- net FX_OUT: now also J4.5 (Pin_5)
- net GND: now also J5.1 (Pin_1)
- net J_IN: now also J4.2 (Pin_2)
- net J_OUT: now also J4.3 (Pin_3)
- net LED: now also J4.6 (Pin_6)
- net VDD: now also J5.3 (Pin_3)
- net WAH_POT: now reaches A1.26 (ADC_4)
- net WAH_POT: now also J5.2 (Pin_2)
- no-connect marks 30 -> 26

Commit message: fix mirror
Parts:
- removed H2: MountingHole_Pad, MountingHole:MountingHole_3.2mm_M3_Pad, symbol Mechanical:MountingHole_Pad
Changed lines of the file:
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@@
-	)
-	(symbol
-		(lib_id "power:GND")
-		(at 328.93 102.87 0)
-		(unit 1)
-		(exclude_from_sim no)
-		(in_bom yes)
-		(on_board yes)
-		(dnp no)
-		(fields_autoplaced yes)
-		(property "Reference" "#PWR031"
-			(at 328.93 109.22 0)
-			(effects
-				(font
-					(size 1.27 1.27)
-				)
-				(hide yes)
-			)
-		)
-		(property "Value" "GND"
-			(at 328.93 107.95 0)
-			(effects
-				(font
-					(size 1.27 1.27)
-				)
-			)
-		)
-		(property "Footprint" ""
-			(at 328.93 102.87 0)
-			(effects
-				(font
-					(size 1.27 1.27)
-				)
-				(hide yes)
-			)
-		)
-		(property "Datasheet" ""
-			(at 328.93 102.87 0)
-			(effects
-				(font
-					(size 1.27 1.27)
-				)
-				(hide yes)
-			)
-		)
-		(property "Description" "Power symbol creates a global label with name \"GND\" , ground"
-			(at 328.93 102.87 0)
-			(effects
-				(font
-					(size 1.27 1.27)
-				)
-				(hide yes)
-			)
-		)
-		(pin "1"
-		)
-		(instances
-			(project "wah"
-				(path "/93d00cbf-8e4b-443f-bc57-0c283a060166"
-					(reference "#PWR031")
-					(unit 1)
-				)
-			)
-		)
 	)
 	(symbol
@@
 					(unit 1)
 				)
-			)
-		)
-	)
-	(symbol
-		(lib_id "Mechanical:MountingHole_Pad")
-		(at 328.93 100.33 0)
-		(unit 1)
-		(exclude_from_sim no)
-		(in_bom no)
-		(on_board yes)
-		(dnp no)
-		(fields_autoplaced yes)
-		(property "Reference" "H2"
-			(at 331.47 97.7899 0)
-			(effects
-				(font
-					(size 1.27 1.27)
-				)
-				(justify left)
-			)
-		)
-		(property "Value" "MountingHole_Pad"
-			(at 331.47 100.3299 0)
-			(effects
-				(font
-					(size 1.27 1.27)
-				)
-				(justify left)
-			)
-		)
-		(property "Footprint" "MountingHole:MountingHole_3.2mm_M3_Pad"
-			(at 328.93 100.33 0)
-			(effects
-				(font
-					(size 1.27 1.27)
-				)
-				(hide yes)
-			)
-		)
-		(property "Datasheet" "~"
-			(at 328.93 100.33 0)
-			(effects
-				(font
-					(size 1.27 1.27)
-				)
-				(hide yes)
-			)
-		)
-		(property "Description" "Mounting Hole with connection"
-			(at 328.93 100.33 0)
-			(effects
-				(font
-					(size 1.27 1.27)
-				)
-				(hide yes)
-			)
-		)
-		(pin "1"
-		)
-		(instances
-			(project "wah"
-				(path "/93d00cbf-8e4b-443f-bc57-0c283a060166"
-					(reference "H2")
-					(unit 1)
-				)

Commit message: improve pcb
Other:
- title: Wah -> BadBaby Wah
- moved on the sheet: J4, J5
Changed lines of the file:
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@@
 	(paper "A3")
 	(title_block
-		(title "Wah")
-		(date "2025-11-13")
-		(rev "0.6.1")
+		(title "BadBaby Wah")
+		(date "2025-11-16")
+		(rev "0.7")
 		(company "KnightHill Engineering")
 	)
@@
 	(wire
 		(pts
-			(xy 299.72 185.42) (xy 300.99 185.42)
+			(xy 288.29 134.62) (xy 289.56 134.62)
 		)
 		(stroke
@@
 	(wire
 		(pts
-			(xy 299.72 187.96) (xy 300.99 187.96)
+			(xy 288.29 137.16) (xy 289.56 137.16)
 		)
 		(stroke
@@
 	(wire
 		(pts
-			(xy 299.72 182.88) (xy 300.99 182.88)
+			(xy 288.29 132.08) (xy 289.56 132.08)
 		)
 		(stroke
@@
 	(wire
 		(pts
-			(xy 297.18 205.74) (xy 300.99 205.74)
+			(xy 285.75 154.94) (xy 289.56 154.94)
 		)
 		(stroke
@@
 	(wire
 		(pts
-			(xy 297.18 207.01) (xy 297.18 205.74)
+			(xy 285.75 156.21) (xy 285.75 154.94)
 		)
 		(stroke
@@
 	(wire
 		(pts
-			(xy 297.18 203.2) (xy 300.99 203.2)
+			(xy 285.75 152.4) (xy 289.56 152.4)
 		)
 		(stroke
@@
 	(wire
 		(pts
-			(xy 299.72 190.5) (xy 300.99 190.5)
+			(xy 288.29 139.7) (xy 289.56 139.7)
 		)
 		(stroke
@@
 	(wire
 		(pts
-			(xy 293.37 177.8) (xy 300.99 177.8)
+			(xy 281.94 127) (xy 289.56 127)
 		)
 		(stroke
@@
 	(wire
 		(pts
-			(xy 297.18 200.66) (xy 300.99 200.66)
+			(xy 285.75 149.86) (xy 289.56 149.86)
 		)
 		(stroke
@@
 	(wire
 		(pts
-			(xy 299.72 180.34) (xy 300.99 180.34)
+			(xy 288.29 129.54) (xy 289.56 129.54)
 		)
 		(stroke
@@
 	)
 	(label "FX_IN"
-		(at 299.72 185.42 180)
+		(at 288.29 134.62 180)
 		(effects
 			(font
@@
 	)
 	(label "J_OUT"
-		(at 299.72 182.88 180)
+		(at 288.29 132.08 180)
 		(effects
 			(font
@@
 	)
 	(label "LED"
-		(at 299.72 190.5 180)
+		(at 288.29 139.7 180)
 		(effects
 			(font
@@
 	)
 	(label "J_IN"
-		(at 299.72 180.34 180)
+		(at 288.29 129.54 180)
 		(effects
 			(font
@@
 	)
 	(label "FX_OUT"
-		(at 299.72 187.96 180)
+		(at 288.29 137.16 180)
 		(effects
 			(font
@@
 	)
 	(label "WAH_POT"
-		(at 297.18 203.2 180)
+		(at 285.75 152.4 180)
 		(effects
 			(font
@@
 	(symbol
 		(lib_id "power:VDD")
-		(at 297.18 207.01 180)
+		(at 285.75 156.21 180)
 		(unit 1)
 		(exclude_from_sim no)
@@
 		(fields_autoplaced yes)
 		(property "Reference" "#PWR033"
-			(at 297.18 203.2 0)
+			(at 285.75 152.4 0)
 			(effects
 				(font
@@
 		)
 		(property "Value" "VDD"
-			(at 297.18 212.09 0)
+			(at 285.75 161.29 0)
 			(effects
 				(font
@@
 		)
 		(property "Footprint" ""
-			(at 297.18 207.01 0)
+			(at 285.75 156.21 0)
 			(effects
 				(font
@@
 		)
 		(property "Datasheet" ""
-			(at 297.18 207.01 0)
+			(at 285.75 156.21 0)
 			(effects
 				(font
@@
 		)
 		(property "Description" "Power symbol creates a global label with name \"VDD\""
-			(at 297.18 207.01 0)
+			(at 285.75 156.21 0)
 			(effects
 				(font
@@
 	(symbol
 		(lib_id "power:GND")
-		(at 297.18 200.66 180)
+		(at 285.75 149.86 180)
 		(unit 1)
 		(exclude_from_sim no)
@@
 		(fields_autoplaced yes)
 		(property "Reference" "#PWR032"
-			(at 297.18 194.31 0)
+			(at 285.75 143.51 0)
 			(effects
 				(font
@@
 		)
 		(property "Value" "GND"
-			(at 297.18 195.58 0)
+			(at 285.75 144.78 0)
 			(effects
 				(font
@@
 		)
 		(property "Footprint" ""
-			(at 297.18 200.66 0)
+			(at 285.75 149.86 0)
 			(effects
 				(font
@@
 		)
 		(property "Datasheet" ""
-			(at 297.18 200.66 0)
+			(at 285.75 149.86 0)
 			(effects
 				(font
@@
 		)
 		(property "Description" "Power symbol creates a global label with name \"GND\" , ground"
-			(at 297.18 200.66 0)
+			(at 285.75 149.86 0)
 			(effects
 				(font
@@
 	(symbol
 		(lib_id "Connector:Conn_01x06_Pin")
-		(at 306.07 182.88 0)
+		(at 294.64 132.08 0)
 		(mirror y)
 		(unit 1)
@@
 		(dnp no)
 		(property "Reference" "J4"
-			(at 305.435 172.72 0)
+			(at 294.005 121.92 0)
 			(effects
 				(font
@@
 		)
 		(property "Value" "Conn_01x06_Pin"
-			(at 305.435 175.26 0)
+			(at 294.005 124.46 0)
 			(effects
 				(font
@@
 		)
 		(property "Footprint" "Connector_PinHeader_2.54mm:PinHeader_1x06_P2.54mm_Vertical"
-			(at 306.07 182.88 0)
+			(at 294.64 132.08 0)
 			(effects
 				(font
@@
 		)
 		(property "Datasheet" "~"
-			(at 306.07 182.88 0)
+			(at 294.64 132.08 0)
 			(effects
 				(font
@@
 		)
 		(property "Description" "Generic connector, single row, 01x06, script generated"
-			(at 306.07 182.88 0)
+			(at 294.64 132.08 0)
 			(effects
 				(font
@@
 	(symbol
 		(lib_id "Connector:Conn_01x03_Pin")
-		(at 306.07 203.2 0)
+		(at 294.64 152.4 0)
 		(mirror y)
 		(unit 1)
@@
 		(dnp no)
 		(property "Reference" "J5"
-			(at 307.34 204.4701 0)
+			(at 295.91 153.6701 0)
 			(effects
 				(font
@@
 		)
 		(property "Value" "Conn_01x03_Pin"
-			(at 307.34 201.9301 0)
+			(at 295.91 151.1301 0)
 			(effects
 				(font
@@
 		)
 		(property "Footprint" "Connector_PinHeader_2.54mm:PinHeader_1x03_P2.54mm_Vertical"
-			(at 306.07 203.2 0)
+			(at 294.64 152.4 0)
 			(effects
 				(font
@@
 		)
 		(property "Datasheet" "~"
-			(at 306.07 203.2 0)
+			(at 294.64 152.4 0)
 			(effects
 				(font
@@
 		)
 		(property "Description" "Generic connector, single row, 01x03, script generated"
-			(at 306.07 203.2 0)
+			(at 294.64 152.4 0)
 			(effects
 				(font
@@
 	(symbol
 		(lib_id "power:+9V")
-		(at 293.37 177.8 90)
+		(at 281.94 127 90)
 		(mirror x)
 		(unit 1)
@@
 		(fields_autoplaced yes)
 		(property "Reference" "#PWR029"
-			(at 297.18 177.8 0)
+			(at 285.75 127 0)
 			(effects
 				(font
@@
 		)
 		(property "Value" "+9V"
-			(at 289.56 177.7999 90)
+			(at 278.13 126.9999 90)
 			(effects
 				(font
@@
 		)
 		(property "Footprint" ""
-			(at 293.37 177.8 0)
+			(at 281.94 127 0)
 			(effects
 				(font
@@
 		)
 		(property "Datasheet" ""
-			(at 293.37 177.8 0)
+			(at 281.94 127 0)
 			(effects
 				(font
@@
 		)
 		(property "Description" "Power symbol creates a global label with name \"+9V\""
-			(at 293.37 177.8 0)
+			(at 281.94 127 0)
 			(effects
 				(font

Commit message: add CB dimention
Parts:
- H1: footprint MountingHole:MountingHole_3.2mm_M3_Pad -> MountingHole:MountingHole_4.5mm_Pad
Changed lines of the file:
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@@
 			)
 		)
-		(property "Footprint" "MountingHole:MountingHole_3.2mm_M3_Pad"
+		(property "Footprint" "MountingHole:MountingHole_4.5mm_Pad"
 			(at 328.93 83.82 0)
 			(effects

Commit message: finalze pcb
Changed lines of the file:
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@@
 				)
 				(justify left)
+				(hide yes)
 			)
 		)
@@
 				)
 				(justify left)
+				(hide yes)
 			)
 		)

Commit message: remove pot 4
Parts:
- removed RV4: 10k, Potentiometer_THT:Potentiometer_Runtron_RM-065_Vertical, symbol Device:R_Potentiometer
- RV1, RV2, RV3: footprint Potentiometer_THT:Potentiometer_Runtron_RM-065_Vertical -> Potentiometer_THT:Potentiometer_Vishay_T73YP_Vertical
Connections:
- net POT4: no longer names the net of A1.25 (ADC_3)
- no-connect marks 26 -> 27

Commit message: add trimmer footprint
Parts:
- RV1, RV2, RV3: footprint Potentiometer_THT:Potentiometer_Vishay_T73YP_Vertical -> CustomFootprints:Trimmer_JBR_3362P
Changed lines of the file:
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@@
 			)
 		)
-		(property "Footprint" "Potentiometer_THT:Potentiometer_Vishay_T73YP_Vertical"
+		(property "Footprint" "CustomFootprints:Trimmer_JBR_3362P"
 			(at 62.23 156.21 0)
 			(effects
@@
 			)
 		)
-		(property "Footprint" "Potentiometer_THT:Potentiometer_Vishay_T73YP_Vertical"
+		(property "Footprint" "CustomFootprints:Trimmer_JBR_3362P"
 			(at 62.23 137.16 0)
 			(effects
@@
 			)
 		)
-		(property "Footprint" "Potentiometer_THT:Potentiometer_Vishay_T73YP_Vertical"
+		(property "Footprint" "CustomFootprints:Trimmer_JBR_3362P"
 			(at 62.23 119.38 0)
 			(effects

Commit message: improve trimmer footprint
Parts:
- RV1, RV2, RV3: footprint CustomFootprints:Trimmer_JBR_3362P -> CustomFootprints:3362P
Changed lines of the file:
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@@
 			)
 		)
-		(property "Footprint" "CustomFootprints:Trimmer_JBR_3362P"
+		(property "Footprint" "CustomFootprints:3362P"
 			(at 62.23 156.21 0)
 			(effects
@@
 			)
 		)
-		(property "Footprint" "CustomFootprints:Trimmer_JBR_3362P"
+		(property "Footprint" "CustomFootprints:3362P"
 			(at 62.23 137.16 0)
 			(effects
@@
 			)
 		)
-		(property "Footprint" "CustomFootprints:Trimmer_JBR_3362P"
+		(property "Footprint" "CustomFootprints:3362P"
 			(at 62.23 119.38 0)
 			(effects
